File: usb_3/usb_3.kicad_sch (KiCad schematic)
At the start: 0 parts

Commit message: working on ams1117
Parts:
- added J1: Power + Data, Connector_USB:USB_C_Receptacle_GCT_USB4105-xx-A_16P_TopMnt_Horizontal, symbol Connector:USB_C_Receptacle
- added J2: Power Only, Connector_USB:USB_C_Receptacle_GCT_USB4105-xx-A_16P_TopMnt_Horizontal, symbol Connector:USB_C_Receptacle
- added J3: USB3_A, Connector_USB:USB3_A_Molex_48393-001, symbol Connector:USB3_A
Connections:
- new net: J1.A10 (RX2-), J1.B10 (RX1-)
- new net: J1.A11 (RX2+), J1.B11 (RX1+)
- new net: J1.A2 (TX1+), J1.B2 (TX2+)
- new net: J1.A3 (TX1-), J1.B3 (TX2-)
- new net: J1.A4 (VBUS), J1.A9 (VBUS), J1.B4 (VBUS), J1.B9 (VBUS)
- new net: J1.A6 (D+), J1.B6 (D+), J3.3 (D+)
- new net: J1.A7 (D-), J1.B7 (D-), J3.2 (D-)
- new net +5V: J2.A4 (VBUS), J2.A9 (VBUS), J2.B4 (VBUS), J2.B9 (VBUS), J3.1 (VBUS)
- new net GND: J1.A1 (GND), J1.A12 (GND), J1.B1 (GND), J1.B12 (GND), J2.A1 (GND), J2.A12 (GND), J2.B1 (GND), J2.B12 (GND), J3.4 (GND)
